File: Hardware/Storage.sch (KiCad schematic (older format))
At the start: 7 parts, among them J3 Micro_SD_Card, Q3 S8550

Commit message: Created PCB file and laid out components
Parts:
- C5, C6: footprint (none) -> Capacitor_SMD:C_0603_1608Metric
- J3: footprint (none) -> Connector_Card:microSD_HC_Hirose_DM3AT-SF-PEJM5
- R11, R12: footprint (none) -> Resistor_SMD:R_0603_1608Metric
- SDLED1: footprint (none) -> LED_SMD:LED_0603_1608Metric
Changed lines of the file:
@@
 F 0 "J3" H 7750 4567 50  0000 C CNN
 F 1 "Micro_SD_Card" H 7750 4476 50  0000 C CNN
-F 2 "" H 8950 4150 50  0001 C CNN
+F 2 "Connector_Card:microSD_HC_Hirose_DM3AT-SF-PEJM5" H 8950 4150 50  0001 C CNN
 F 3 "http://katalog.we-online.de/em/datasheet/693072010801.pdf" H 7800 3850 50  0001 C CNN
 	1    7800 3850
@@
 F 0 "C6" H 6192 4046 50  0000 L CNN
 F 1 "10uF" H 6192 3955 50  0000 L CNN
-F 2 "" H 6100 4000 50  0001 C CNN
+F 2 "Capacitor_SMD:C_0603_1608Metric" H 6100 4000 50  0001 C CNN
 F 3 "~" H 6100 4000 50  0001 C CNN
 	1    6100 4000
@@
 F 0 "C5" H 5842 4046 50  0000 L CNN
 F 1 "0.1uF" H 5842 3955 50  0000 L CNN
-F 2 "" H 5750 4000 50  0001 C CNN
+F 2 "Capacitor_SMD:C_0603_1608Metric" H 5750 4000 50  0001 C CNN
 F 3 "~" H 5750 4000 50  0001 C CNN
 	1    5750 4000
@@
 F 0 "SDLED1" H 4493 3545 50  0000 C CNN
 F 1 "LED" H 4493 3636 50  0000 C CNN
-F 2 "" H 4500 3800 50  0001 C CNN
+F 2 "LED_SMD:LED_0603_1608Metric" H 4500 3800 50  0001 C CNN
 F 3 "~" H 4500 3800 50  0001 C CNN
 	1    4500 3800
@@
 F 0 "R12" V 3954 3800 50  0000 C CNN
 F 1 "1k" V 4045 3800 50  0000 C CNN
-F 2 "" H 4150 3800 50  0001 C CNN
+F 2 "Resistor_SMD:R_0603_1608Metric" H 4150 3800 50  0001 C CNN
 F 3 "~" H 4150 3800 50  0001 C CNN
 	1    4150 3800
@@
 F 0 "R11" H 3641 4254 50  0000 R CNN
 F 1 "12k" H 3641 4345 50  0000 R CNN
-F 2 "" H 3700 4300 50  0001 C CNN
+F 2 "Resistor_SMD:R_0603_1608Metric" H 3700 4300 50  0001 C CNN
 F 3 "~" H 3700 4300 50  0001 C CNN
 	1    3700 4300
