File: Hardware/usb.sch (KiCad schematic (older format))
At the start: 13 parts

Commit message: Added circuitry to program ESP32
Connections:
- net VBUS: now also D?.4 (K)
- net RTS: now reaches U?.19 (RTS)
- net DTR: now reaches U?.23 (DTR)
- no-connect marks 11 -> 9
Other:
- moved on the sheet: D?
Changed lines of the file:
@@
 P 6150 2750
 AR Path="/60872B38" Ref="#PWR?"  Part="1"
-AR Path="/608652D9/60872B38" Ref="#PWR?"  Part="1"
-F 0 "#PWR?" H 6150 2600 50  0001 C CNN
+AR Path="/608652D9/60872B38" Ref="#PWR0115"  Part="1"
+F 0 "#PWR0115" H 6150 2600 50  0001 C CNN
 F 1 "+3V3" H 6165 2923 50  0000 C CNN
 F 2 "" H 6150 2750 50  0001 C CNN
@@
 	6800 2850 6850 2850
 $Comp
-L power:+3V3 #PWR?
+L power:+3V3 #PWR0116
 U 1 1 60872B3F
 P 6850 2200
-F 0 "#PWR?" H 6850 2050 50  0001 C CNN
+F 0 "#PWR0116" H 6850 2050 50  0001 C CNN
 F 1 "+3V3" H 6865 2373 50  0000 C CNN
 F 2 "" H 6850 2200 50  0001 C CNN
@@
 	7350 2600 7250 2600
 $Comp
-L power:GND #PWR?
+L power:GND #PWR0117
 U 1 1 60872B57
 P 7350 2600
-F 0 "#PWR?" H 7350 2350 50  0001 C CNN
+F 0 "#PWR0117" H 7350 2350 50  0001 C CNN
 F 1 "GND" H 7355 2427 50  0000 C CNN
 F 2 "" H 7350 2600 50  0001 C CNN
@@
 	6850 2850 6900 2850
 NoConn ~ 7500 3250
-NoConn ~ 7500 3350
 NoConn ~ 7500 3650
-NoConn ~ 7500 3750
 NoConn ~ 7500 3850
 NoConn ~ 7500 4150
@@
 P 8400 4300
 AR Path="/60872B6B" Ref="#PWR?"  Part="1"
-AR Path="/608652D9/60872B6B" Ref="#PWR?"  Part="1"
-F 0 "#PWR?" H 8400 4150 50  0001 C CNN
+AR Path="/608652D9/60872B6B" Ref="#PWR0118"  Part="1"
+F 0 "#PWR0118" H 8400 4150 50  0001 C CNN
 F 1 "+3V3" H 8415 4473 50  0000 C CNN
 F 2 "" H 8400 4300 50  0001 C CNN
@@
 P 6950 4750
 AR Path="/60872BE4" Ref="#PWR?"  Part="1"
-AR Path="/608652D9/60872BE4" Ref="#PWR?"  Part="1"
-F 0 "#PWR?" H 6950 4500 50  0001 C CNN
+AR Path="/608652D9/60872BE4" Ref="#PWR0119"  Part="1"
+F 0 "#PWR0119" H 6950 4500 50  0001 C CNN
 F 1 "GND" H 6955 4577 50  0000 C CNN
 F 2 "" H 6950 4750 50  0001 C CNN
@@
 P 3600 4650
 AR Path="/60872BF8" Ref="#PWR?"  Part="1"
-AR Path="/608652D9/60872BF8" Ref="#PWR?"  Part="1"
-F 0 "#PWR?" H 3600 4400 50  0001 C CNN
+AR Path="/608652D9/60872BF8" Ref="#PWR0120"  Part="1"
+F 0 "#PWR0120" H 3600 4400 50  0001 C CNN
 F 1 "GND" H 3605 4477 50  0000 C CNN
 F 2 "" H 3600 4650 50  0001 C CNN
@@
 P 4850 3650
 AR Path="/60883C5B" Ref="#PWR?"  Part="1"
-AR Path="/608652D9/60883C5B" Ref="#PWR?"  Part="1"
-F 0 "#PWR?" H 4850 3400 50  0001 C CNN
+AR Path="/608652D9/60883C5B" Ref="#PWR0121"  Part="1"
+F 0 "#PWR0121" H 4850 3400 50  0001 C CNN
 F 1 "GND" H 4855 3477 50  0000 C CNN
 F 2 "" H 4850 3650 50  0001 C CNN
@@
 P 5750 4400
 AR Path="/608A68DE" Ref="#PWR?"  Part="1"
-AR Path="/608652D9/608A68DE" Ref="#PWR?"  Part="1"
-F 0 "#PWR?" H 5750 4150 50  0001 C CNN
+AR Path="/608652D9/608A68DE" Ref="#PWR0122"  Part="1"
+F 0 "#PWR0122" H 5750 4150 50  0001 C CNN
 F 1 "GND" H 5755 4227 50  0000 C CNN
 F 2 "" H 5750 4400 50  0001 C CNN
@@
 Wire Wire Line
 	4850 3300 4850 3350
-Text Label 4850 5550 0    50   ~ 0
+Text Label 4800 5400 0    50   ~ 0
 D+
-Text Label 4850 5450 0    50   ~ 0
+Text Label 4800 5300 0    50   ~ 0
 D-
-Text Label 5350 4850 0    50   ~ 0
+Text Label 4800 5200 0    50   ~ 0
 VBUS
 $Comp
 L power:GND #PWR?
 U 1 1 608CFC5E
-P 5500 5450
+P 5450 5300
 AR Path="/608CFC5E" Ref="#PWR?"  Part="1"
-AR Path="/608652D9/608CFC5E" Ref="#PWR?"  Part="1"
-F 0 "#PWR?" H 5500 5200 50  0001 C CNN
-F 1 "GND" V 5505 5322 50  0000 R CNN
-F 2 "" H 5500 5450 50  0001 C CNN
-F 3 "" H 5500 5450 50  0001 C CNN
-	1    5500 5450
+AR Path="/608652D9/608CFC5E" Ref="#PWR0123"  Part="1"
+F 0 "#PWR0123" H 5450 5050 50  0001 C CNN
+F 1 "GND" V 5455 5172 50  0000 R CNN
+F 2 "" H 5450 5300 50  0001 C CNN
+F 3 "" H 5450 5300 50  0001 C CNN
+	1    5450 5300
 	0    -1   -1   0
 $EndComp
@@
 L Power_Protection:SP0503BAHT D?
 U 1 1 608FE2F6
-P 5250 5450
-F 0 "D?" V 5592 5450 50  0000 C CNN
-F 1 "SP0503BAHT" V 5501 5450 50  0000 C CNN
-F 2 "Package_TO_SOT_SMD:SOT-143" H 5475 5400 50  0001 L CNN
-F 3 "http://www.littelfuse.com/~/media/files/littelfuse/technical%20resources/documents/data%20sheets/sp05xxba.pdf" H 5375 5575 50  0001 C CNN
-	1    5250 5450
+P 5200 5300
+F 0 "D?" V 5542 5300 50  0000 C CNN
+F 1 "SP0503BAHT" V 5451 5300 50  0000 C CNN
+F 2 "Package_TO_SOT_SMD:SOT-143" H 5425 5250 50  0001 L CNN
+F 3 "http://www.littelfuse.com/~/media/files/littelfuse/technical%20resources/documents/data%20sheets/sp05xxba.pdf" H 5325 5425 50  0001 C CNN
+	1    5200 5300
 	0    -1   -1   0
 $EndComp
 Wire Wire Line
-	5450 5450 5500 5450
-Wire Wire Line
-	4850 5350 5050 5350
-Wire Wire Line
-	4850 5450 5050 5450
-Wire Wire Line
-	4850 5550 5050 5550
+	5400 5300 5450 5300
+Wire Wire Line
+	4800 5200 5000 5200
+Wire Wire Line
+	4800 5300 5000 5300
+Wire Wire Line
+	4800 5400 5000 5400
+Wire Wire Line
+	7500 3350 7650 3350
+Wire Wire Line
+	7500 3750 7650 3750
+Text HLabel 7650 3350 2    50   Output ~ 0
+RTS
+Text HLabel 7650 3750 2    50   Output ~ 0
+DTR
 $EndSCHEMATC

Commit message: Manually merged power to main
Might have some problems with USB
Parts:
- P?: symbol Connector:USB_C_Plug_USB2.0 -> VLAD-rescue:USB_C_Plug_USB2.0-Connector
Changed lines of the file:
@@
 EESchema Schematic File Version 4
+LIBS:VLAD-cache
 EELAYER 30 0
 EELAYER END
 $Descr A4 11693 8268
 encoding utf-8
-Sheet 4 4
+Sheet 4 5
 Title ""
 Date ""
@@
 	3450 4600 3450 4650
 $Comp
-L Connector:USB_C_Plug_USB2.0 P?
+L VLAD-rescue:USB_C_Plug_USB2.0-Connector P?
 U 1 1 60872C01
 P 3750 3700
