File: Hardware/usb.sch (KiCad schematic (older format))
At the start: 17 parts

Commit message: Fixed some of the ERC errors
Parts:
- gave numbers to parts that had none: 17
Changed lines of the file:
@@
 P 6150 2750
 AR Path="/60872B38" Ref="#PWR?"  Part="1"
-AR Path="/608652D9/60872B38" Ref="#PWR0115"  Part="1"
-F 0 "#PWR0115" H 6150 2600 50  0001 C CNN
+AR Path="/608652D9/60872B38" Ref="#PWR030"  Part="1"
+F 0 "#PWR030" H 6150 2600 50  0001 C CNN
 F 1 "+3V3" H 6165 2923 50  0000 C CNN
 F 2 "" H 6150 2750 50  0001 C CNN
@@
 	6800 2850 6850 2850
 $Comp
-L power:+3V3 #PWR0116
+L power:+3V3 #PWR031
 U 1 1 60872B3F
 P 6850 2200
-F 0 "#PWR0116" H 6850 2050 50  0001 C CNN
+F 0 "#PWR031" H 6850 2050 50  0001 C CNN
 F 1 "+3V3" H 6865 2373 50  0000 C CNN
 F 2 "" H 6850 2200 50  0001 C CNN
@@
 P 7150 2250
 AR Path="/60872B45" Ref="C?"  Part="1"
-AR Path="/608652D9/60872B45" Ref="C?"  Part="1"
-F 0 "C?" V 6921 2250 50  0000 C CNN
+AR Path="/608652D9/60872B45" Ref="C9"  Part="1"
+F 0 "C9" V 6921 2250 50  0000 C CNN
 F 1 "4.7uF" V 7012 2250 50  0000 C CNN
 F 2 "" H 7150 2250 50  0001 C CNN
@@
 $EndComp
 $Comp
-L Device:C_Small C?
+L Device:C_Small C10
 U 1 1 60872B4B
 P 7150 2600
-F 0 "C?" V 6921 2600 50  0000 C CNN
+F 0 "C10" V 6921 2600 50  0000 C CNN
 F 1 "0.1uF" V 7012 2600 50  0000 C CNN
 F 2 "" H 7150 2600 50  0001 C CNN
@@
 	7350 2600 7250 2600
 $Comp
-L power:GND #PWR0117
+L power:GND #PWR033
 U 1 1 60872B57
 P 7350 2600
-F 0 "#PWR0117" H 7350 2350 50  0001 C CNN
+F 0 "#PWR033" H 7350 2350 50  0001 C CNN
 F 1 "GND" H 7355 2427 50  0000 C CNN
 F 2 "" H 7350 2600 50  0001 C CNN
@@
 P 8400 4300
 AR Path="/60872B6B" Ref="#PWR?"  Part="1"
-AR Path="/608652D9/60872B6B" Ref="#PWR0118"  Part="1"
-F 0 "#PWR0118" H 8400 4150 50  0001 C CNN
+AR Path="/608652D9/60872B6B" Ref="#PWR034"  Part="1"
+F 0 "#PWR034" H 8400 4150 50  0001 C CNN
 F 1 "+3V3" H 8415 4473 50  0000 C CNN
 F 2 "" H 8400 4300 50  0001 C CNN
@@
 P 8050 4600
 AR Path="/60872B78" Ref="R?"  Part="1"
-AR Path="/608652D9/60872B78" Ref="R?"  Part="1"
-F 0 "R?" V 7854 4600 50  0000 C CNN
+AR Path="/608652D9/60872B78" Ref="R20"  Part="1"
+F 0 "R20" V 7854 4600 50  0000 C CNN
 F 1 "1k" V 7945 4600 50  0000 C CNN
 F 2 "" H 8050 4600 50  0001 C CNN
@@
 P 8050 4250
 AR Path="/60872B7E" Ref="R?"  Part="1"
-AR Path="/608652D9/60872B7E" Ref="R?"  Part="1"
-F 0 "R?" V 7854 4250 50  0000 C CNN
+AR Path="/608652D9/60872B7E" Ref="R19"  Part="1"
+F 0 "R19" V 7854 4250 50  0000 C CNN
 F 1 "1k" V 7945 4250 50  0000 C CNN
 F 2 "" H 8050 4250 50  0001 C CNN
@@
 P 6900 3750
 AR Path="/60872B86" Ref="U?"  Part="1"
-AR Path="/608652D9/60872B86" Ref="U?"  Part="1"
-F 0 "U?" H 6900 4831 50  0000 C CNN
+AR Path="/608652D9/60872B86" Ref="U3"  Part="1"
+F 0 "U3" H 6900 4831 50  0000 C CNN
 F 1 "CP2102N-A01-GQFN24" H 6900 4740 50  0000 C CNN
 F 2 "Package_DFN_QFN:QFN-24-1EP_4x4mm_P0.5mm_EP2.6x2.6mm" H 7350 2950 50  0001 L CNN
@@
 P 7800 4600
 AR Path="/60872B8D" Ref="TxLED?"  Part="1"
-AR Path="/608652D9/60872B8D" Ref="TxLED?"  Part="1"
-F 0 "TxLED?" H 7793 4817 50  0000 C CNN
+AR Path="/608652D9/60872B8D" Ref="TxLED1"  Part="1"
+F 0 "TxLED1" H 7793 4817 50  0000 C CNN
 F 1 "LED" H 7793 4726 50  0000 C CNN
 F 2 "" H 7800 4600 50  0001 C CNN
@@
 P 7800 4250
 AR Path="/60872B93" Ref="RxLED?"  Part="1"
-AR Path="/608652D9/60872B93" Ref="RxLED?"  Part="1"
-F 0 "RxLED?" H 7793 4467 50  0000 C CNN
+AR Path="/608652D9/60872B93" Ref="RxLED1"  Part="1"
+F 0 "RxLED1" H 7793 4467 50  0000 C CNN
 F 1 "LED" H 7793 4376 50  0000 C CNN
 F 2 "" H 7800 4250 50  0001 C CNN
@@
 P 5750 4200
 AR Path="/60872BAC" Ref="R?"  Part="1"
-AR Path="/608652D9/60872BAC" Ref="R?"  Part="1"
-F 0 "R?" H 5691 4154 50  0000 R CNN
+AR Path="/608652D9/60872BAC" Ref="R17"  Part="1"
+F 0 "R17" H 5691 4154 50  0000 R CNN
 F 1 "47.5k" H 5691 4245 50  0000 R CNN
 F 2 "" H 5750 4200 50  0001 C CNN
@@
 P 5500 4050
 AR Path="/60872BB2" Ref="R?"  Part="1"
-AR Path="/608652D9/60872BB2" Ref="R?"  Part="1"
-F 0 "R?" V 5696 4050 50  0000 C CNN
+AR Path="/608652D9/60872BB2" Ref="R16"  Part="1"
+F 0 "R16" V 5696 4050 50  0000 C CNN
 F 1 "22.1k" V 5605 4050 50  0000 C CNN
 F 2 "" H 5500 4050 50  0001 C CNN
@@
 P 6950 4750
 AR Path="/60872BE4" Ref="#PWR?"  Part="1"
-AR Path="/608652D9/60872BE4" Ref="#PWR0119"  Part="1"
-F 0 "#PWR0119" H 6950 4500 50  0001 C CNN
+AR Path="/608652D9/60872BE4" Ref="#PWR032"  Part="1"
+F 0 "#PWR032" H 6950 4500 50  0001 C CNN
 F 1 "GND" H 6955 4577 50  0000 C CNN
 F 2 "" H 6950 4750 50  0001 C CNN
@@
 P 6150 2950
 AR Path="/60872BEE" Ref="R?"  Part="1"
-AR Path="/608652D9/60872BEE" Ref="R?"  Part="1"
-F 0 "R?" H 6209 2996 50  0000 L CNN
+AR Path="/608652D9/60872BEE" Ref="R18"  Part="1"
+F 0 "R18" H 6209 2996 50  0000 L CNN
 F 1 "1k" H 6209 2905 50  0000 L CNN
 F 2 "" H 6150 2950 50  0001 C CNN
@@
 P 3600 4650
 AR Path="/60872BF8" Ref="#PWR?"  Part="1"
-AR Path="/608652D9/60872BF8" Ref="#PWR0120"  Part="1"
-F 0 "#PWR0120" H 3600 4400 50  0001 C CNN
+AR Path="/608652D9/60872BF8" Ref="#PWR026"  Part="1"
+F 0 "#PWR026" H 3600 4400 50  0001 C CNN
 F 1 "GND" H 3605 4477 50  0000 C CNN
 F 2 "" H 3600 4650 50  0001 C CNN
@@
 P 3750 3700
 AR Path="/60872C01" Ref="P?"  Part="1"
-AR Path="/608652D9/60872C01" Ref="P?"  Part="1"
-F 0 "P?" H 3857 4567 50  0000 C CNN
+AR Path="/608652D9/60872C01" Ref="P1"  Part="1"
+F 0 "P1" H 3857 4567 50  0000 C CNN
 F 1 "USB_C_Plug_USB2.0" H 3857 4476 50  0000 C CNN
 F 2 "Connector_USB:USB_C_Receptacle_GCT_USB4085" H 3900 3700 50  0001 C CNN
@@
 P 4850 3650
 AR Path="/60883C5B" Ref="#PWR?"  Part="1"
-AR Path="/608652D9/60883C5B" Ref="#PWR0121"  Part="1"
-F 0 "#PWR0121" H 4850 3400 50  0001 C CNN
+AR Path="/608652D9/60883C5B" Ref="#PWR027"  Part="1"
+F 0 "#PWR027" H 4850 3400 50  0001 C CNN
 F 1 "GND" H 4855 3477 50  0000 C CNN
 F 2 "" H 4850 3650 50  0001 C CNN
@@
 P 4850 3450
 AR Path="/608840CF" Ref="R?"  Part="1"
-AR Path="/608652D9/608840CF" Ref="R?"  Part="1"
-F 0 "R?" H 4791 3404 50  0000 R CNN
+AR Path="/608652D9/608840CF" Ref="R15"  Part="1"
+F 0 "R15" H 4791 3404 50  0000 R CNN
 F 1 "5.1k" H 4791 3495 50  0000 R CNN
 F 2 "" H 4850 3450 50  0001 C CNN
@@
 P 5750 4400
 AR Path="/608A68DE" Ref="#PWR?"  Part="1"
-AR Path="/608652D9/608A68DE" Ref="#PWR0122"  Part="1"
-F 0 "#PWR0122" H 5750 4150 50  0001 C CNN
+AR Path="/608652D9/608A68DE" Ref="#PWR029"  Part="1"
+F 0 "#PWR029" H 5750 4150 50  0001 C CNN
 F 1 "GND" H 5755 4227 50  0000 C CNN
 F 2 "" H 5750 4400 50  0001 C CNN
@@
 P 5450 5300
 AR Path="/608CFC5E" Ref="#PWR?"  Part="1"
-AR Path="/608652D9/608CFC5E" Ref="#PWR0123"  Part="1"
-F 0 "#PWR0123" H 5450 5050 50  0001 C CNN
+AR Path="/608652D9/608CFC5E" Ref="#PWR028"  Part="1"
+F 0 "#PWR028" H 5450 5050 50  0001 C CNN
 F 1 "GND" V 5455 5172 50  0000 R CNN
 F 2 "" H 5450 5300 50  0001 C CNN
@@
 NoConn ~ 6300 3550
 $Comp
-L Power_Protection:SP0503BAHT D?
+L Power_Protection:SP0503BAHT D1
 U 1 1 608FE2F6
 P 5200 5300
-F 0 "D?" V 5542 5300 50  0000 C CNN
+F 0 "D1" V 5542 5300 50  0000 C CNN
 F 1 "SP0503BAHT" V 5451 5300 50  0000 C CNN
 F 2 "Package_TO_SOT_SMD:SOT-143" H 5425 5250 50  0001 L CNN
@@
 DTR
 $Comp
-L Connector:TestPoint TP?
+L Connector:TestPoint TP8
 U 1 1 607C08D3
 P 9200 2850
-F 0 "TP?" V 9154 3038 50  0000 L CNN
+F 0 "TP8" V 9154 3038 50  0000 L CNN
 F 1 "TestPoint" V 9245 3038 50  0000 L CNN
 F 2 "" H 9400 2850 50  0001 C CNN
@@
 $EndComp
 $Comp
-L Connector:TestPoint TP?
+L Connector:TestPoint TP9
 U 1 1 607C0C71
 P 9200 3050
-F 0 "TP?" V 9154 3238 50  0000 L CNN
+F 0 "TP9" V 9154 3238 50  0000 L CNN
 F 1 "TestPoint" V 9245 3238 50  0000 L CNN
 F 2 "" H 9400 3050 50  0001 C CNN
@@
 	9200 3050 9050 3050
 $Comp
-L Connector:TestPoint TP?
+L Connector:TestPoint TP10
 U 1 1 607C5A06
 P 9200 3250
-F 0 "TP?" V 9154 3438 50  0000 L CNN
+F 0 "TP10" V 9154 3438 50  0000 L CNN
 F 1 "TestPoint" V 9245 3438 50  0000 L CNN
 F 2 "" H 9400 3250 50  0001 C CNN
@@
 	9200 3250 9050 3250
 $Comp
-L Connector:TestPoint TP?
+L Connector:TestPoint TP11
 U 1 1 607C6B8E
 P 9200 3450
-F 0 "TP?" V 9154 3638 50  0000 L CNN
+F 0 "TP11" V 9154 3638 50  0000 L CNN
 F 1 "TestPoint" V 9245 3638 50  0000 L CNN
 F 2 "" H 9400 3450 50  0001 C CNN
@@
 Text HLabel 9050 3450 0    50   Output ~ 0
 DTR
+$Comp
+L power:PWR_FLAG #FLG0103
+U 1 1 608936C2
+P 4350 3100
+F 0 "#FLG0103" H 4350 3175 50  0001 C CNN
+F 1 "PWR_FLAG" H 4350 3273 50  0000 C CNN
+F 2 "" H 4350 3100 50  0001 C CNN
+F 3 "~" H 4350 3100 50  0001 C CNN
+	1    4350 3100
+	1    0    0    -1
+$EndComp
+Connection ~ 4350 3100
 $EndSCHEMATC

Commit message: Created PCB file and laid out components
Parts:
- C10, C9: footprint (none) -> Capacitor_SMD:C_0603_1608Metric
- R15, R16, R17, R18, R19, R20: footprint (none) -> Resistor_SMD:R_0603_1608Metric
- RxLED1, TxLED1: footprint (none) -> LED_SMD:LED_0603_1608Metric
- TP10, TP11, TP8, TP9: footprint (none) -> TestPoint:TestPoint_THTPad_1.5x1.5mm_Drill0.7mm
Changed lines of the file:
@@
 F 0 "C9" V 6921 2250 50  0000 C CNN
 F 1 "4.7uF" V 7012 2250 50  0000 C CNN
-F 2 "" H 7150 2250 50  0001 C CNN
+F 2 "Capacitor_SMD:C_0603_1608Metric" H 7150 2250 50  0001 C CNN
 F 3 "~" H 7150 2250 50  0001 C CNN
 	1    7150 2250
@@
 F 0 "C10" V 6921 2600 50  0000 C CNN
 F 1 "0.1uF" V 7012 2600 50  0000 C CNN
-F 2 "" H 7150 2600 50  0001 C CNN
+F 2 "Capacitor_SMD:C_0603_1608Metric" H 7150 2600 50  0001 C CNN
 F 3 "~" H 7150 2600 50  0001 C CNN
 	1    7150 2600
@@
 F 0 "R20" V 7854 4600 50  0000 C CNN
 F 1 "1k" V 7945 4600 50  0000 C CNN
-F 2 "" H 8050 4600 50  0001 C CNN
+F 2 "Resistor_SMD:R_0603_1608Metric" H 8050 4600 50  0001 C CNN
 F 3 "~" H 8050 4600 50  0001 C CNN
 	1    8050 4600
@@
 F 0 "R19" V 7854 4250 50  0000 C CNN
 F 1 "1k" V 7945 4250 50  0000 C CNN
-F 2 "" H 8050 4250 50  0001 C CNN
+F 2 "Resistor_SMD:R_0603_1608Metric" H 8050 4250 50  0001 C CNN
 F 3 "~" H 8050 4250 50  0001 C CNN
 	1    8050 4250
@@
 F 0 "TxLED1" H 7793 4817 50  0000 C CNN
 F 1 "LED" H 7793 4726 50  0000 C CNN
-F 2 "" H 7800 4600 50  0001 C CNN
+F 2 "LED_SMD:LED_0603_1608Metric" H 7800 4600 50  0001 C CNN
 F 3 "~" H 7800 4600 50  0001 C CNN
 	1    7800 4600
@@
 F 0 "RxLED1" H 7793 4467 50  0000 C CNN
 F 1 "LED" H 7793 4376 50  0000 C CNN
-F 2 "" H 7800 4250 50  0001 C CNN
+F 2 "LED_SMD:LED_0603_1608Metric" H 7800 4250 50  0001 C CNN
 F 3 "~" H 7800 4250 50  0001 C CNN
 	1    7800 4250
@@
 F 0 "R17" H 5691 4154 50  0000 R CNN
 F 1 "47.5k" H 5691 4245 50  0000 R CNN
-F 2 "" H 5750 4200 50  0001 C CNN
+F 2 "Resistor_SMD:R_0603_1608Metric" H 5750 4200 50  0001 C CNN
 F 3 "~" H 5750 4200 50  0001 C CNN
 	1    5750 4200
@@
 F 0 "R16" V 5696 4050 50  0000 C CNN
 F 1 "22.1k" V 5605 4050 50  0000 C CNN
-F 2 "" H 5500 4050 50  0001 C CNN
+F 2 "Resistor_SMD:R_0603_1608Metric" H 5500 4050 50  0001 C CNN
 F 3 "~" H 5500 4050 50  0001 C CNN
 	1    5500 4050
@@
 F 0 "R18" H 6209 2996 50  0000 L CNN
 F 1 "1k" H 6209 2905 50  0000 L CNN
-F 2 "" H 6150 2950 50  0001 C CNN
+F 2 "Resistor_SMD:R_0603_1608Metric" H 6150 2950 50  0001 C CNN
 F 3 "~" H 6150 2950 50  0001 C CNN
 	1    6150 2950
@@
 F 0 "R15" H 4791 3404 50  0000 R CNN
 F 1 "5.1k" H 4791 3495 50  0000 R CNN
-F 2 "" H 4850 3450 50  0001 C CNN
+F 2 "Resistor_SMD:R_0603_1608Metric" H 4850 3450 50  0001 C CNN
 F 3 "~" H 4850 3450 50  0001 C CNN
 	1    4850 3450
@@
 F 0 "TP8" V 9154 3038 50  0000 L CNN
 F 1 "TestPoint" V 9245 3038 50  0000 L CNN
-F 2 "" H 9400 2850 50  0001 C CNN
+F 2 "TestPoint:TestPoint_THTPad_1.5x1.5mm_Drill0.7mm" H 9400 2850 50  0001 C CNN
 F 3 "~" H 9400 2850 50  0001 C CNN
 	1    9200 2850
@@
 F 0 "TP9" V 9154 3238 50  0000 L CNN
 F 1 "TestPoint" V 9245 3238 50  0000 L CNN
-F 2 "" H 9400 3050 50  0001 C CNN
+F 2 "TestPoint:TestPoint_THTPad_1.5x1.5mm_Drill0.7mm" H 9400 3050 50  0001 C CNN
 F 3 "~" H 9400 3050 50  0001 C CNN
 	1    9200 3050
@@
 F 0 "TP10" V 9154 3438 50  0000 L CNN
 F 1 "TestPoint" V 9245 3438 50  0000 L CNN
-F 2 "" H 9400 3250 50  0001 C CNN
+F 2 "TestPoint:TestPoint_THTPad_1.5x1.5mm_Drill0.7mm" H 9400 3250 50  0001 C CNN
 F 3 "~" H 9400 3250 50  0001 C CNN
 	1    9200 3250
@@
 F 0 "TP11" V 9154 3638 50  0000 L CNN
 F 1 "TestPoint" V 9245 3638 50  0000 L CNN
-F 2 "" H 9400 3450 50  0001 C CNN
+F 2 "TestPoint:TestPoint_THTPad_1.5x1.5mm_Drill0.7mm" H 9400 3450 50  0001 C CNN
 F 3 "~" H 9400 3450 50  0001 C CNN
 	1    9200 3450

Commit message: Genuine Confusion
Changed to an ideal diode whatever tf that is
Parts:
- P1: symbol Connector:USB_C_Plug_USB2.0 -> VLAD-rescue:USB_C_Plug_USB2.0-Connector
Changed lines of the file:
@@
 EESchema Schematic File Version 4
+LIBS:VLAD-cache
 EELAYER 30 0
 EELAYER END
@@
 	3450 4600 3450 4650
 $Comp
-L Connector:USB_C_Plug_USB2.0 P?
+L VLAD-rescue:USB_C_Plug_USB2.0-Connector P?
 U 1 1 60872C01
 P 3750 3700
