File: Hardware/VLAD.sch (KiCad schematic (older format))
At the start: 29 parts, among them J1 BMP388, J2 BNO055, Q1 S8050, Q2 S8050, SW1 SW_Push, SW2 SW_Push, U1 ESP32-WROOM-32

Commit message: Created PCB file and laid out components
Parts:
- BZ1: footprint (none) -> Connector_PinHeader_2.54mm:PinHeader_2x01_P2.54mm_Vertical
- C1, C2, C3, C4: footprint (none) -> Capacitor_SMD:C_0603_1608Metric
- J1: footprint (none) -> Connector_PinHeader_2.54mm:PinHeader_1x08_P2.54mm_Vertical
- J2: footprint (none) -> Connector_PinSocket_2.54mm:PinSocket_1x06_P2.54mm_Vertical
- R1, R10, R2, R3, R4, R5, R6, R7, R8, R9: footprint (none) -> Resistor_SMD:R_0603_1608Metric
- SW1, SW2: footprint (none) -> Button_Switch_SMD:SW_Push_1P1T_NO_6x6mm_H9.5mm
- TP1, TP2, TP3, TP4, TP5, TP6, TP7: footprint (none) -> TestPoint:TestPoint_THTPad_1.5x1.5mm_Drill0.7mm
Changed lines of the file:
@@
 F 0 "C3" V 6221 1750 50  0000 C CNN
 F 1 "10uF" V 6312 1750 50  0000 C CNN
-F 2 "" H 6450 1750 50  0001 C CNN
+F 2 "Capacitor_SMD:C_0603_1608Metric" H 6450 1750 50  0001 C CNN
 F 3 "~" H 6450 1750 50  0001 C CNN
 	1    6450 1750
@@
 F 0 "C4" V 6221 2100 50  0000 C CNN
 F 1 "0.1uF" V 6312 2100 50  0000 C CNN
-F 2 "" H 6450 2100 50  0001 C CNN
+F 2 "Capacitor_SMD:C_0603_1608Metric" H 6450 2100 50  0001 C CNN
 F 3 "~" H 6450 2100 50  0001 C CNN
 	1    6450 2100
@@
 F 0 "R1" H 1809 5546 50  0000 L CNN
 F 1 "12k" H 1809 5455 50  0000 L CNN
-F 2 "" H 1750 5500 50  0001 C CNN
+F 2 "Resistor_SMD:R_0603_1608Metric" H 1750 5500 50  0001 C CNN
 F 3 "~" H 1750 5500 50  0001 C CNN
 	1    1750 5500
@@
 F 0 "R9" H 7609 2996 50  0000 L CNN
 F 1 "5k" H 7609 2905 50  0000 L CNN
-F 2 "" H 7550 2950 50  0001 C CNN
+F 2 "Resistor_SMD:R_0603_1608Metric" H 7550 2950 50  0001 C CNN
 F 3 "~" H 7550 2950 50  0001 C CNN
 	1    7550 2950
@@
 F 0 "R2" V 1704 4100 50  0000 C CNN
 F 1 "1k" V 1795 4100 50  0000 C CNN
-F 2 "" H 1900 4100 50  0001 C CNN
+F 2 "Resistor_SMD:R_0603_1608Metric" H 1900 4100 50  0001 C CNN
 F 3 "~" H 1900 4100 50  0001 C CNN
 	1    1900 4100
@@
 F 0 "R3" V 1704 4800 50  0000 C CNN
 F 1 "1k" V 1795 4800 50  0000 C CNN
-F 2 "" H 1900 4800 50  0001 C CNN
+F 2 "Resistor_SMD:R_0603_1608Metric" H 1900 4800 50  0001 C CNN
 F 3 "~" H 1900 4800 50  0001 C CNN
 	1    1900 4800
@@
 F 0 "R5" H 2259 5546 50  0000 L CNN
 F 1 "5k" H 2259 5455 50  0000 L CNN
-F 2 "" H 2200 5500 50  0001 C CNN
+F 2 "Resistor_SMD:R_0603_1608Metric" H 2200 5500 50  0001 C CNN
 F 3 "~" H 2200 5500 50  0001 C CNN
 	1    2200 5500
@@
 F 0 "SW1" H 1450 6485 50  0000 C CNN
 F 1 "SW_Push" H 1450 6394 50  0000 C CNN
-F 2 "" H 1450 6400 50  0001 C CNN
+F 2 "Button_Switch_SMD:SW_Push_1P1T_NO_6x6mm_H9.5mm" H 1450 6400 50  0001 C CNN
 F 3 "~" H 1450 6400 50  0001 C CNN
 	1    1450 6200
@@
 F 0 "R4" V 1704 6200 50  0000 C CNN
 F 1 "470" V 1795 6200 50  0000 C CNN
-F 2 "" H 1900 6200 50  0001 C CNN
+F 2 "Resistor_SMD:R_0603_1608Metric" H 1900 6200 50  0001 C CNN
 F 3 "~" H 1900 6200 50  0001 C CNN
 	1    1900 6200
@@
 F 0 "C2" V 2421 6500 50  0000 C CNN
 F 1 "1uF" V 2512 6500 50  0000 C CNN
-F 2 "" H 2650 6500 50  0001 C CNN
+F 2 "Capacitor_SMD:C_0603_1608Metric" H 2650 6500 50  0001 C CNN
 F 3 "~" H 2650 6500 50  0001 C CNN
 	1    2650 6500
@@
 F 0 "R8" V 2904 6200 50  0000 C CNN
 F 1 "470" V 2995 6200 50  0000 C CNN
-F 2 "" H 3100 6200 50  0001 C CNN
+F 2 "Resistor_SMD:R_0603_1608Metric" H 3100 6200 50  0001 C CNN
 F 3 "~" H 3100 6200 50  0001 C CNN
 	1    3100 6200
@@
 F 0 "SW2" H 2650 6485 50  0000 C CNN
 F 1 "SW_Push" H 2650 6394 50  0000 C CNN
-F 2 "" H 2650 6400 50  0001 C CNN
+F 2 "Button_Switch_SMD:SW_Push_1P1T_NO_6x6mm_H9.5mm" H 2650 6400 50  0001 C CNN
 F 3 "~" H 2650 6400 50  0001 C CNN
 	1    2650 6200
@@
 F 0 "C1" V 1221 6500 50  0000 C CNN
 F 1 "1nF" V 1312 6500 50  0000 C CNN
-F 2 "" H 1450 6500 50  0001 C CNN
+F 2 "Capacitor_SMD:C_0603_1608Metric" H 1450 6500 50  0001 C CNN
 F 3 "~" H 1450 6500 50  0001 C CNN
 	1    1450 6500
@@
 F 0 "TP3" V 2454 1288 50  0000 L CNN
 F 1 "TestPoint" V 2545 1288 50  0000 L CNN
-F 2 "" H 2700 1100 50  0001 C CNN
+F 2 "TestPoint:TestPoint_THTPad_1.5x1.5mm_Drill0.7mm" H 2700 1100 50  0001 C CNN
 F 3 "~" H 2700 1100 50  0001 C CNN
 	1    2500 1100
@@
 F 0 "TP5" V 2454 1688 50  0000 L CNN
 F 1 "TestPoint" V 2545 1688 50  0000 L CNN
-F 2 "" H 2700 1500 50  0001 C CNN
+F 2 "TestPoint:TestPoint_THTPad_1.5x1.5mm_Drill0.7mm" H 2700 1500 50  0001 C CNN
 F 3 "~" H 2700 1500 50  0001 C CNN
 	1    2500 1500
@@
 F 0 "TP4" V 2454 1488 50  0000 L CNN
 F 1 "TestPoint" V 2545 1488 50  0000 L CNN
-F 2 "" H 2700 1300 50  0001 C CNN
+F 2 "TestPoint:TestPoint_THTPad_1.5x1.5mm_Drill0.7mm" H 2700 1300 50  0001 C CNN
 F 3 "~" H 2700 1300 50  0001 C CNN
 	1    2500 1300
@@
 F 0 "TP6" V 2454 1888 50  0000 L CNN
 F 1 "TestPoint" V 2545 1888 50  0000 L CNN
-F 2 "" H 2700 1700 50  0001 C CNN
+F 2 "TestPoint:TestPoint_THTPad_1.5x1.5mm_Drill0.7mm" H 2700 1700 50  0001 C CNN
 F 3 "~" H 2700 1700 50  0001 C CNN
 	1    2500 1700
@@
 F 0 "TP7" V 2454 2088 50  0000 L CNN
 F 1 "TestPoint" V 2545 2088 50  0000 L CNN
-F 2 "" H 2700 1900 50  0001 C CNN
+F 2 "TestPoint:TestPoint_THTPad_1.5x1.5mm_Drill0.7mm" H 2700 1900 50  0001 C CNN
 F 3 "~" H 2700 1900 50  0001 C CNN
 	1    2500 1900
@@
 F 0 "TP1" V 1854 7238 50  0000 L CNN
 F 1 "TestPoint" V 1945 7238 50  0000 L CNN
-F 2 "" H 2100 7050 50  0001 C CNN
+F 2 "TestPoint:TestPoint_THTPad_1.5x1.5mm_Drill0.7mm" H 2100 7050 50  0001 C CNN
 F 3 "~" H 2100 7050 50  0001 C CNN
 	1    1900 7050
@@
 F 0 "TP2" V 1854 7438 50  0000 L CNN
 F 1 "TestPoint" V 1945 7438 50  0000 L CNN
-F 2 "" H 2100 7250 50  0001 C CNN
+F 2 "TestPoint:TestPoint_THTPad_1.5x1.5mm_Drill0.7mm" H 2100 7250 50  0001 C CNN
 F 3 "~" H 2100 7250 50  0001 C CNN
 	1    1900 7250
@@
 F 0 "R6" V 2354 2600 50  0000 C CNN
 F 1 "10k" V 2445 2600 50  0000 C CNN
-F 2 "" H 2550 2600 50  0001 C CNN
+F 2 "Resistor_SMD:R_0603_1608Metric" H 2550 2600 50  0001 C CNN
 F 3 "~" H 2550 2600 50  0001 C CNN
 	1    2550 2600
@@
 F 0 "R7" V 2354 2900 50  0000 C CNN
 F 1 "10k" V 2445 2900 50  0000 C CNN
-F 2 "" H 2550 2900 50  0001 C CNN
+F 2 "Resistor_SMD:R_0603_1608Metric" H 2550 2900 50  0001 C CNN
 F 3 "~" H 2550 2900 50  0001 C CNN
 	1    2550 2900
@@
 F 0 "BZ1" V 9101 4863 50  0000 R CNN
 F 1 "Buzzer" V 9010 4863 50  0000 R CNN
-F 2 "" V 9025 5150 50  0001 C CNN
+F 2 "Connector_PinHeader_2.54mm:PinHeader_2x01_P2.54mm_Vertical" V 9025 5150 50  0001 C CNN
 F 3 "~" V 9025 5150 50  0001 C CNN
 	1    9050 5050
@@
 F 0 "R10" V 8504 5200 50  0000 C CNN
 F 1 "R_Small" V 8595 5200 50  0000 C CNN
-F 2 "" H 8700 5200 50  0001 C CNN
+F 2 "Resistor_SMD:R_0603_1608Metric" H 8700 5200 50  0001 C CNN
 F 3 "~" H 8700 5200 50  0001 C CNN
 	1    8700 5200
@@
 F 0 "J2" H 9378 3376 50  0000 L CNN
 F 1 "BNO055" H 9378 3285 50  0000 L CNN
-F 2 "" H 9350 3400 50  0001 C CNN
+F 2 "Connector_PinSocket_2.54mm:PinSocket_1x06_P2.54mm_Vertical" H 9350 3400 50  0001 C CNN
 F 3 "~" H 9350 3400 50  0001 C CNN
 	1    9350 3400
@@
 F 0 "J1" H 9378 2426 50  0000 L CNN
 F 1 "BMP388" H 9378 2335 50  0000 L CNN
-F 2 "" H 9350 2450 50  0001 C CNN
+F 2 "Connector_PinHeader_2.54mm:PinHeader_1x08_P2.54mm_Vertical" H 9350 2450 50  0001 C CNN
 F 3 "~" H 9350 2450 50  0001 C CNN
 	1    9350 2450

Commit message: Final changes for this first draft
Parts:
- J1: footprint Connector_PinHeader_2.54mm:PinHeader_1x08_P2.54mm_Vertical -> Connector_PinSocket_2.54mm:PinSocket_1x08_P2.54mm_Vertical
Changed lines of the file:
@@
 F 0 "J1" H 9378 2426 50  0000 L CNN
 F 1 "BMP388" H 9378 2335 50  0000 L CNN
-F 2 "Connector_PinHeader_2.54mm:PinHeader_1x08_P2.54mm_Vertical" H 9350 2450 50  0001 C CNN
+F 2 "Connector_PinSocket_2.54mm:PinSocket_1x08_P2.54mm_Vertical" H 9350 2450 50  0001 C CNN
 F 3 "~" H 9350 2450 50  0001 C CNN
 	1    9350 2450
