File: Hardware/PowerCircuitry.sch (KiCad schematic (older format))
At the start: 29 parts, among them J4 Conn_01x02_Male, Q5 MMBT3904, Q6 MMBT3904, SW3 SW_SPST, U4 MAX40200AUK

Commit message: Changed 300uF to 4x68uF
Cos why not
Parts:
- removed C1.2, C2.2: 300uF, Capacitor_SMD:C_0603_1608Metric, symbol Device:CP1
- added C1.? (x8): 68uF, Capacitor_THT:CP_Radial_D6.3mm_P2.50mm, symbol Device:CP1
- C1.1, C2.1: footprint Capacitor_SMD:C_0603_1608Metric -> Capacitor_THT:CP_Radial_D6.3mm_P2.50mm
Connections:
- wire segments 80 -> 102
Other:
- moved on the sheet: D2, D3
Changed lines of the file:
@@
 L Device:D_Schottky D2
 U 1 1 607B6B59
-P 4100 750
-F 0 "D2" H 4100 966 50  0000 C CNN
-F 1 "D_Schottky" H 4100 875 50  0000 C CNN
-F 2 "Diode_SMD:D_0603_1608Metric" H 4100 750 50  0001 C CNN
-F 3 "~" H 4100 750 50  0001 C CNN
-	1    4100 750
-	-1   0    0    1
-$EndComp
-Wire Wire Line
-	3950 750  3950 1250
-Connection ~ 3950 1250
+P 3950 1000
+F 0 "D2" H 3950 1216 50  0000 C CNN
+F 1 "D_Schottky" H 3950 1125 50  0000 C CNN
+F 2 "Diode_SMD:D_0603_1608Metric" H 3950 1000 50  0001 C CNN
+F 3 "~" H 3950 1000 50  0001 C CNN
+	1    3950 1000
+	0    1    1    0
+$EndComp
 $Comp
 L Device:CP1 C1.1
@@
 F 0 "C1.1" H 3065 1446 50  0000 L CNN
 F 1 "68uF" H 3065 1355 50  0000 L CNN
-F 2 "Capacitor_SMD:C_0603_1608Metric" H 2950 1400 50  0001 C CNN
+F 2 "Capacitor_THT:CP_Radial_D6.3mm_P2.50mm" H 2950 1400 50  0001 C CNN
 F 3 "~" H 2950 1400 50  0001 C CNN
 	1    2950 1400
@@
 $EndComp
 $Comp
-L Device:CP1 C1.2
-U 1 1 607B8269
-P 4450 900
-F 0 "C1.2" H 4565 946 50  0000 L CNN
-F 1 "300uF" H 4565 855 50  0000 L CNN
-F 2 "Capacitor_SMD:C_0603_1608Metric" H 4450 900 50  0001 C CNN
-F 3 "~" H 4450 900 50  0001 C CNN
-	1    4450 900
-	1    0    0    -1
-$EndComp
-Wire Wire Line
-	4250 750  4450 750
-$Comp
 L power:GND #PWR044
 U 1 1 607B9113
-P 4450 1050
-F 0 "#PWR044" H 4450 800 50  0001 C CNN
-F 1 "GND" H 4455 877 50  0000 C CNN
-F 2 "" H 4450 1050 50  0001 C CNN
-F 3 "" H 4450 1050 50  0001 C CNN
-	1    4450 1050
+P 4550 1150
+F 0 "#PWR044" H 4550 900 50  0001 C CNN
+F 1 "GND" H 4555 977 50  0000 C CNN
+F 2 "" H 4550 1150 50  0001 C CNN
+F 3 "" H 4550 1150 50  0001 C CNN
+	1    4550 1150
 	1    0    0    -1
 $EndComp
@@
 $EndComp
 Wire Wire Line
-	4450 750  4950 750
-Wire Wire Line
 	4950 750  4950 950
 Wire Wire Line
 	4950 950  5200 950
-Connection ~ 4450 750
 $Comp
 L power:GND #PWR047
@@
 Wire Wire Line
 	4950 750  6950 750
-Connection ~ 4950 750
 $Comp
 L Device:R RSense1
@@
 F 0 "C2.1" H 3065 3946 50  0000 L CNN
 F 1 "68uF" H 3065 3855 50  0000 L CNN
-F 2 "Capacitor_SMD:C_0603_1608Metric" H 2950 3900 50  0001 C CNN
+F 2 "Capacitor_THT:CP_Radial_D6.3mm_P2.50mm" H 2950 3900 50  0001 C CNN
 F 3 "~" H 2950 3900 50  0001 C CNN
 	1    2950 3900
@@
 L Device:D_Schottky D3
 U 1 1 607D4386
-P 4100 3250
-F 0 "D3" H 4100 3466 50  0000 C CNN
-F 1 "D_Schottky" H 4100 3375 50  0000 C CNN
-F 2 "Diode_SMD:D_0603_1608Metric" H 4100 3250 50  0001 C CNN
-F 3 "~" H 4100 3250 50  0001 C CNN
-	1    4100 3250
-	-1   0    0    1
-$EndComp
-Wire Wire Line
-	3950 3750 3950 3250
-Connection ~ 3950 3750
-$Comp
-L Device:CP1 C2.2
-U 1 1 607D5B4D
-P 4450 3400
-F 0 "C2.2" H 4565 3446 50  0000 L CNN
-F 1 "300uF" H 4565 3355 50  0000 L CNN
-F 2 "Capacitor_SMD:C_0603_1608Metric" H 4450 3400 50  0001 C CNN
-F 3 "~" H 4450 3400 50  0001 C CNN
-	1    4450 3400
-	1    0    0    -1
-$EndComp
-Wire Wire Line
-	4250 3250 4450 3250
+P 3950 3500
+F 0 "D3" H 3950 3716 50  0000 C CNN
+F 1 "D_Schottky" H 3950 3625 50  0000 C CNN
+F 2 "Diode_SMD:D_0603_1608Metric" H 3950 3500 50  0001 C CNN
+F 3 "~" H 3950 3500 50  0001 C CNN
+	1    3950 3500
+	0    1    1    0
+$EndComp
 $Comp
 L Device:C C2.3
@@
 $EndComp
 Wire Wire Line
-	4450 3250 4950 3250
-Wire Wire Line
 	4950 3250 4950 3450
 Wire Wire Line
 	4950 3450 5200 3450
-Connection ~ 4450 3250
 $Comp
 L power:GND #PWR048
@@
 Wire Wire Line
 	4950 3250 6700 3250
-Connection ~ 4950 3250
 Wire Wire Line
 	4950 3450 4950 4000
@@
 L power:GND #PWR045
 U 1 1 607EA56C
-P 4450 3550
-F 0 "#PWR045" H 4450 3300 50  0001 C CNN
-F 1 "GND" H 4455 3377 50  0000 C CNN
-F 2 "" H 4450 3550 50  0001 C CNN
-F 3 "" H 4450 3550 50  0001 C CNN
-	1    4450 3550
+P 4500 3650
+F 0 "#PWR045" H 4500 3400 50  0001 C CNN
+F 1 "GND" H 4505 3477 50  0000 C CNN
+F 2 "" H 4500 3650 50  0001 C CNN
+F 3 "" H 4500 3650 50  0001 C CNN
+	1    4500 3650
 	1    0    0    -1
 $EndComp
@@
 	1    0    0    -1
 $EndComp
+Wire Wire Line
+	2050 3750 2050 4250
+Wire Wire Line
+	2050 4250 1500 4250
+Wire Wire Line
+	1500 4250 1500 4500
+Wire Wire Line
+	2300 4750 2300 3750
+Wire Wire Line
+	2300 3750 2450 3750
+$Comp
+L power:GND #PWR0101
+U 1 1 60A25E03
+P 1900 5150
+F 0 "#PWR0101" H 1900 4900 50  0001 C CNN
+F 1 "GND" H 1905 4977 50  0000 C CNN
+F 2 "" H 1900 5150 50  0001 C CNN
+F 3 "" H 1900 5150 50  0001 C CNN
+	1    1900 5150
+	1    0    0    -1
+$EndComp
+Wire Wire Line
+	3950 1150 3950 1250
+Connection ~ 3950 1250
+Wire Wire Line
+	3950 850  3950 750
+Connection ~ 4950 750
+$Comp
+L Device:CP1 C1.?
+U 1 1 60A60441
+P 4450 900
+F 0 "C1.?" H 4565 946 50  0000 L CNN
+F 1 "68uF" H 4565 855 50  0000 L CNN
+F 2 "Capacitor_THT:CP_Radial_D6.3mm_P2.50mm" H 4450 900 50  0001 C CNN
+F 3 "~" H 4450 900 50  0001 C CNN
+	1    4450 900
+	1    0    0    -1
+$EndComp
+$Comp
+L Device:CP1 C1.?
+U 1 1 60A60F44
+P 4650 900
+F 0 "C1.?" H 4765 946 50  0000 L CNN
+F 1 "68uF" H 4765 855 50  0000 L CNN
+F 2 "Capacitor_THT:CP_Radial_D6.3mm_P2.50mm" H 4650 900 50  0001 C CNN
+F 3 "~" H 4650 900 50  0001 C CNN
+	1    4650 900
+	1    0    0    -1
+$EndComp
+$Comp
+L Device:CP1 C1.?
+U 1 1 60A613E6
+P 4850 900
+F 0 "C1.?" H 4965 946 50  0000 L CNN
+F 1 "68uF" H 4965 855 50  0000 L CNN
+F 2 "Capacitor_THT:CP_Radial_D6.3mm_P2.50mm" H 4850 900 50  0001 C CNN
+F 3 "~" H 4850 900 50  0001 C CNN
+	1    4850 900
+	1    0    0    -1
+$EndComp
+Connection ~ 4850 750
+Wire Wire Line
+	4850 750  4950 750
+Connection ~ 4650 750
+Wire Wire Line
+	4650 750  4850 750
+Connection ~ 4450 750
+Wire Wire Line
+	4450 750  4650 750
+Wire Wire Line
+	3950 750  4250 750
+$Comp
+L Device:CP1 C1.?
+U 1 1 60A668C7
+P 4250 900
+F 0 "C1.?" H 4365 946 50  0000 L CNN
+F 1 "68uF" H 4365 855 50  0000 L CNN
+F 2 "Capacitor_THT:CP_Radial_D6.3mm_P2.50mm" H 4250 900 50  0001 C CNN
+F 3 "~" H 4250 900 50  0001 C CNN
+	1    4250 900
+	1    0    0    -1
+$EndComp
+Connection ~ 4250 750
+Wire Wire Line
+	4250 750  4450 750
+Wire Wire Line
+	4250 1050 4450 1050
+Connection ~ 4450 1050
+Wire Wire Line
+	4450 1050 4550 1050
+Connection ~ 4650 1050
+Wire Wire Line
+	4650 1050 4850 1050
+Wire Wire Line
+	4550 1150 4550 1050
+Connection ~ 4550 1050
+Wire Wire Line
+	4550 1050 4650 1050
 $Comp
 L Analog_Switch:MAX40200AUK U4
@@
 $EndComp
 Wire Wire Line
-	2050 3750 2050 4250
-Wire Wire Line
-	2050 4250 1500 4250
-Wire Wire Line
-	1500 4250 1500 4750
-Wire Wire Line
-	2300 4750 2300 3750
-Wire Wire Line
-	2300 3750 2450 3750
-$Comp
-L power:GND #PWR0101
-U 1 1 60A25E03
-P 1900 5150
-F 0 "#PWR0101" H 1900 4900 50  0001 C CNN
-F 1 "GND" H 1905 4977 50  0000 C CNN
-F 2 "" H 1900 5150 50  0001 C CNN
-F 3 "" H 1900 5150 50  0001 C CNN
-	1    1900 5150
-	1    0    0    -1
-$EndComp
-$Comp
-L power:GND #PWR0102
-U 1 1 60A2712E
-P 1500 4950
-F 0 "#PWR0102" H 1500 4700 50  0001 C CNN
-F 1 "GND" H 1505 4777 50  0000 C CNN
-F 2 "" H 1500 4950 50  0001 C CNN
-F 3 "" H 1500 4950 50  0001 C CNN
-	1    1500 4950
-	1    0    0    -1
-$EndComp
+	1500 4500 1200 4500
+Wire Wire Line
+	1200 4500 1200 4950
+Wire Wire Line
+	1200 4950 1500 4950
+Connection ~ 1500 4500
+Wire Wire Line
+	1500 4500 1500 4750
+Wire Wire Line
+	3950 3650 3950 3750
+Connection ~ 3950 3750
+Wire Wire Line
+	3950 3350 3950 3250
+Wire Wire Line
+	3950 3250 4200 3250
+Connection ~ 4950 3250
+$Comp
+L Device:CP1 C1.?
+U 1 1 60A97AFD
+P 4800 3400
+F 0 "C1.?" H 4915 3446 50  0000 L CNN
+F 1 "68uF" H 4915 3355 50  0000 L CNN
+F 2 "Capacitor_THT:CP_Radial_D6.3mm_P2.50mm" H 4800 3400 50  0001 C CNN
+F 3 "~" H 4800 3400 50  0001 C CNN
+	1    4800 3400
+	1    0    0    -1
+$EndComp
+Connection ~ 4800 3250
+Wire Wire Line
+	4800 3250 4950 3250
+$Comp
+L Device:CP1 C1.?
+U 1 1 60A993A5
+P 4600 3400
+F 0 "C1.?" H 4715 3446 50  0000 L CNN
+F 1 "68uF" H 4715 3355 50  0000 L CNN
+F 2 "Capacitor_THT:CP_Radial_D6.3mm_P2.50mm" H 4600 3400 50  0001 C CNN
+F 3 "~" H 4600 3400 50  0001 C CNN
+	1    4600 3400
+	1    0    0    -1
+$EndComp
+Connection ~ 4600 3250
+Wire Wire Line
+	4600 3250 4800 3250
+$Comp
+L Device:CP1 C1.?
+U 1 1 60A997C6
+P 4400 3400
+F 0 "C1.?" H 4515 3446 50  0000 L CNN
+F 1 "68uF" H 4515 3355 50  0000 L CNN
+F 2 "Capacitor_THT:CP_Radial_D6.3mm_P2.50mm" H 4400 3400 50  0001 C CNN
+F 3 "~" H 4400 3400 50  0001 C CNN
+	1    4400 3400
+	1    0    0    -1
+$EndComp
+Connection ~ 4400 3250
+Wire Wire Line
+	4400 3250 4600 3250
+$Comp
+L Device:CP1 C1.?
+U 1 1 60A99BF5
+P 4200 3400
+F 0 "C1.?" H 4315 3446 50  0000 L CNN
+F 1 "68uF" H 4315 3355 50  0000 L CNN
+F 2 "Capacitor_THT:CP_Radial_D6.3mm_P2.50mm" H 4200 3400 50  0001 C CNN
+F 3 "~" H 4200 3400 50  0001 C CNN
+	1    4200 3400
+	1    0    0    -1
+$EndComp
+Connection ~ 4200 3250
+Wire Wire Line
+	4200 3250 4400 3250
+Wire Wire Line
+	4200 3550 4400 3550
+Connection ~ 4400 3550
+Wire Wire Line
+	4400 3550 4500 3550
+Connection ~ 4600 3550
+Wire Wire Line
+	4600 3550 4800 3550
+Wire Wire Line
+	4500 3650 4500 3550
+Connection ~ 4500 3550
+Wire Wire Line
+	4500 3550 4600 3550
 $EndSCHEMATC

Commit message: Split PCB setup
Setup the PCB with each section split. J5 didn't have a schematic so I picked one.
Parts:
- gave numbers to parts that had none: 8
Changed lines of the file:
@@
 EESchema Schematic File Version 4
-LIBS:VLAD-cache
 EELAYER 30 0
 EELAYER END
@@
 Connection ~ 4950 750
 $Comp
-L Device:CP1 C1.?
+L Device:CP1 C1.7
 U 1 1 60A60441
 P 4450 900
-F 0 "C1.?" H 4565 946 50  0000 L CNN
+F 0 "C1.7" H 4565 946 50  0000 L CNN
 F 1 "68uF" H 4565 855 50  0000 L CNN
 F 2 "Capacitor_THT:CP_Radial_D6.3mm_P2.50mm" H 4450 900 50  0001 C CNN
@@
 $EndComp
 $Comp
-L Device:CP1 C1.?
+L Device:CP1 C1.9
 U 1 1 60A60F44
 P 4650 900
-F 0 "C1.?" H 4765 946 50  0000 L CNN
+F 0 "C1.9" H 4765 946 50  0000 L CNN
 F 1 "68uF" H 4765 855 50  0000 L CNN
 F 2 "Capacitor_THT:CP_Radial_D6.3mm_P2.50mm" H 4650 900 50  0001 C CNN
@@
 $EndComp
 $Comp
-L Device:CP1 C1.?
+L Device:CP1 C1.11
 U 1 1 60A613E6
 P 4850 900
-F 0 "C1.?" H 4965 946 50  0000 L CNN
+F 0 "C1.11" H 4965 946 50  0000 L CNN
 F 1 "68uF" H 4965 855 50  0000 L CNN
 F 2 "Capacitor_THT:CP_Radial_D6.3mm_P2.50mm" H 4850 900 50  0001 C CNN
@@
 	3950 750  4250 750
 $Comp
-L Device:CP1 C1.?
+L Device:CP1 C1.5
 U 1 1 60A668C7
 P 4250 900
-F 0 "C1.?" H 4365 946 50  0000 L CNN
+F 0 "C1.5" H 4365 946 50  0000 L CNN
 F 1 "68uF" H 4365 855 50  0000 L CNN
 F 2 "Capacitor_THT:CP_Radial_D6.3mm_P2.50mm" H 4250 900 50  0001 C CNN
@@
 Connection ~ 4950 3250
 $Comp
-L Device:CP1 C1.?
+L Device:CP1 C1.10
 U 1 1 60A97AFD
 P 4800 3400
-F 0 "C1.?" H 4915 3446 50  0000 L CNN
+F 0 "C1.10" H 4915 3446 50  0000 L CNN
 F 1 "68uF" H 4915 3355 50  0000 L CNN
 F 2 "Capacitor_THT:CP_Radial_D6.3mm_P2.50mm" H 4800 3400 50  0001 C CNN
@@
 	4800 3250 4950 3250
 $Comp
-L Device:CP1 C1.?
+L Device:CP1 C1.8
 U 1 1 60A993A5
 P 4600 3400
-F 0 "C1.?" H 4715 3446 50  0000 L CNN
+F 0 "C1.8" H 4715 3446 50  0000 L CNN
 F 1 "68uF" H 4715 3355 50  0000 L CNN
 F 2 "Capacitor_THT:CP_Radial_D6.3mm_P2.50mm" H 4600 3400 50  0001 C CNN
@@
 	4600 3250 4800 3250
 $Comp
-L Device:CP1 C1.?
+L Device:CP1 C1.6
 U 1 1 60A997C6
 P 4400 3400
-F 0 "C1.?" H 4515 3446 50  0000 L CNN
+F 0 "C1.6" H 4515 3446 50  0000 L CNN
 F 1 "68uF" H 4515 3355 50  0000 L CNN
 F 2 "Capacitor_THT:CP_Radial_D6.3mm_P2.50mm" H 4400 3400 50  0001 C CNN
@@
 	4400 3250 4600 3250
 $Comp
-L Device:CP1 C1.?
+L Device:CP1 C1.2
 U 1 1 60A99BF5
 P 4200 3400
-F 0 "C1.?" H 4315 3446 50  0000 L CNN
+F 0 "C1.2" H 4315 3446 50  0000 L CNN
 F 1 "68uF" H 4315 3355 50  0000 L CNN
 F 2 "Capacitor_THT:CP_Radial_D6.3mm_P2.50mm" H 4200 3400 50  0001 C CNN

Commit message: Fixed some footprints
Things to bring up:
1. Used a 2N2219 BJT (?) transistor for the sake of circuit connection and footprint. IRL would be using either a 2N2222 (which Palash has in stock) or the one linked on the excel sheet.
2. Used a resistor to break 3.3V bus from the node to prevent wrong connections. IRL will just use a breadboard wire to bridge it, unless more elegant ways of doing this. 
3. Need to sort out the global connection bs idk how to do that.
Parts:
- added Q7: 2N2219, Package_TO_SOT_THT:TO-92_Inline, symbol Transistor_BJT:2N2219
- added R21: R, Resistor_THT:R_Axial_DIN0204_L3.6mm_D1.6mm_P1.90mm_Vertical, symbol Device:R
- D2, D3: footprint Diode_SMD:D_0603_1608Metric -> Diode_THT:D_DO-34_SOD68_P7.62mm_Horizontal
- L1, L2: footprint Inductor_SMD:L_0603_1608Metric -> Inductor_THT:L_Toroid_Vertical_L16.0mm_W8.0mm_P7.62mm
- SW3: footprint Button_Switch_SMD:SW_DIP_SPSTx01_Slide_9.78x4.72mm_W8.61mm_P2.54mm -> Button_Switch_THT:SW_DIP_SPSTx01_Slide_9.78x4.72mm_W7.62mm_P2.54mm
Connections:
- net labels added: 12VBusSwitch
- wire segments 102 -> 104
Changed lines of the file:
@@
 EESchema Schematic File Version 4
+LIBS:VLAD-cache
 EELAYER 30 0
 EELAYER END
@@
 F 0 "L1" V 3490 1250 50  0000 C CNN
 F 1 "22uH" V 3399 1250 50  0000 C CNN
-F 2 "Inductor_SMD:L_0603_1608Metric" H 3300 1250 50  0001 C CNN
+F 2 "Inductor_THT:L_Toroid_Vertical_L16.0mm_W8.0mm_P7.62mm" H 3300 1250 50  0001 C CNN
 F 3 "~" H 3300 1250 50  0001 C CNN
 	1    3300 1250
@@
 F 0 "D2" H 3950 1216 50  0000 C CNN
 F 1 "D_Schottky" H 3950 1125 50  0000 C CNN
-F 2 "Diode_SMD:D_0603_1608Metric" H 3950 1000 50  0001 C CNN
+F 2 "Diode_THT:D_DO-34_SOD68_P7.62mm_Horizontal" H 3950 1000 50  0001 C CNN
 F 3 "~" H 3950 1000 50  0001 C CNN
 	1    3950 1000
@@
 F 0 "L2" V 3490 3750 50  0000 C CNN
 F 1 "22uH" V 3399 3750 50  0000 C CNN
-F 2 "Inductor_SMD:L_0603_1608Metric" H 3300 3750 50  0001 C CNN
+F 2 "Inductor_THT:L_Toroid_Vertical_L16.0mm_W8.0mm_P7.62mm" H 3300 3750 50  0001 C CNN
 F 3 "~" H 3300 3750 50  0001 C CNN
 	1    3300 3750
@@
 F 0 "D3" H 3950 3716 50  0000 C CNN
 F 1 "D_Schottky" H 3950 3625 50  0000 C CNN
-F 2 "Diode_SMD:D_0603_1608Metric" H 3950 3500 50  0001 C CNN
+F 2 "Diode_THT:D_DO-34_SOD68_P7.62mm_Horizontal" H 3950 3500 50  0001 C CNN
 F 3 "~" H 3950 3500 50  0001 C CNN
 	1    3950 3500
@@
 	4450 5500 3700 5500
 Connection ~ 2950 3750
-Wire Wire Line
-	2450 1250 2950 1250
 Connection ~ 2450 3750
 Wire Wire Line
 	2450 3750 2950 3750
-Connection ~ 2950 1250
 Wire Wire Line
 	2450 3750 2450 6500
@@
 Wire Wire Line
 	1500 3750 2050 3750
-Wire Wire Line
-	2450 1250 2450 3750
 $Comp
 L Mechanical:MountingHole_Pad H1
@@
 	1    0    0    -1
 $EndComp
-Wire Wire Line
-	2450 6500 3200 6500
 Connection ~ 1100 3750
 $Comp
@@
 F 0 "SW3" H 1300 3985 50  0000 C CNN
 F 1 "SW_SPST" H 1300 3894 50  0000 C CNN
-F 2 "Button_Switch_SMD:SW_DIP_SPSTx01_Slide_9.78x4.72mm_W8.61mm_P2.54mm" H 1300 3750 50  0001 C CNN
+F 2 "Button_Switch_THT:SW_DIP_SPSTx01_Slide_9.78x4.72mm_W7.62mm_P2.54mm" H 1300 3750 50  0001 C CNN
 F 3 "~" H 1300 3750 50  0001 C CNN
 	1    1300 3750
@@
 Wire Wire Line
 	4500 3550 4600 3550
+$Comp
+L Transistor_BJT:2N2219 Q7
+U 1 1 60A91052
+P 2550 3250
+F 0 "Q7" H 2741 3204 50  0000 L CNN
+F 1 "2N2219" H 2741 3295 50  0000 L CNN
+F 2 "Package_TO_SOT_THT:TO-92_Inline" H 2750 3175 50  0001 L CIN
+F 3 "http://www.onsemi.com/pub_link/Collateral/2N2219-D.PDF" H 2550 3250 50  0001 L CNN
+	1    2550 3250
+	-1   0    0    1
+$EndComp
+Wire Wire Line
+	2450 3450 2450 3750
+Wire Wire Line
+	2450 3050 2450 1250
+Wire Wire Line
+	2450 1250 2950 1250
+Connection ~ 2950 1250
+Text GLabel 2750 3250 2    50   Input ~ 0
+12VBusSwitch
+$Comp
+L Device:R R21
+U 1 1 60AA8F0F
+P 2800 6500
+F 0 "R21" V 2593 6500 50  0000 C CNN
+F 1 "R" V 2684 6500 50  0000 C CNN
+F 2 "Resistor_THT:R_Axial_DIN0204_L3.6mm_D1.6mm_P1.90mm_Vertical" V 2730 6500 50  0001 C CNN
+F 3 "~" H 2800 6500 50  0001 C CNN
+	1    2800 6500
+	0    1    1    0
+$EndComp
+Wire Wire Line
+	2450 6500 2650 6500
+Wire Wire Line
+	2950 6500 3200 6500
 $EndSCHEMATC

Commit message: Fixed N-Channel MOSFET, etc
And a few net label tings
Parts:
- removed Q5, Q6: MMBT3904, Package_TO_SOT_SMD:SOT-23, symbol Transistor_BJT:MMBT3904
- added Q? (x2): MTP3055VL, TO254P483X1016X2222-3P, symbol MTP3055VL:MTP3055VL
Connections:
- net labels added: Drain1, Drain2, Gate1, Gate2, Source1, Source2
Changed lines of the file:
@@
-$EndComp
-$Comp
-L Transistor_BJT:MMBT3904 Q5
-U 1 1 607D48DD
-P 4150 1850
-F 0 "Q5" V 4478 1850 50  0000 C CNN
-F 1 "MMBT3904" V 4387 1850 50  0000 C CNN
-F 2 "Package_TO_SOT_SMD:SOT-23" H 4350 1775 50  0001 L CIN
-F 3 "https://www.fairchildsemi.com/datasheets/2N/2N3904.pdf" H 4150 1850 50  0001 L CNN
-	1    4150 1850
-	0    -1   -1   0
-$EndComp
-$Comp
-L Transistor_BJT:MMBT3904 Q6
-U 1 1 607E1E71
-P 4150 4350
-F 0 "Q6" V 4478 4350 50  0000 C CNN
-F 1 "MMBT3904" V 4387 4350 50  0000 C CNN
-F 2 "Package_TO_SOT_SMD:SOT-23" H 4350 4275 50  0001 L CIN
-F 3 "https://www.fairchildsemi.com/datasheets/2N/2N3904.pdf" H 4150 4350 50  0001 L CNN
-	1    4150 4350
-	0    -1   -1   0
 $EndComp
 $Comp
@@
 Wire Wire Line
 	2950 6500 3200 6500
+$Comp
+L MTP3055VL:MTP3055VL Q?
+U 1 1 60AA2630
+P 1400 1500
+F 0 "Q?" H 1400 1770 50  0000 C CNN
+F 1 "MTP3055VL" H 1400 1679 50  0000 C CNN
+F 2 "TO254P483X1016X2222-3P" H 1400 1500 50  0001 L BNN
+F 3 "" H 1400 1500 50  0001 L BNN
+F 4 "MTP3055VL" H 1400 1500 50  0001 L BNN "MPN"
+F 5 "18C7756" H 1400 1500 50  0001 L BNN "OC_NEWARK"
+F 6 "1845563" H 1400 1500 50  0001 L BNN "OC_FARNELL"
+F 7 "Fairchild" H 1400 1500 50  0001 L BNN "SUPPLIER"
+F 8 "TO-220" H 1400 1500 50  0001 L BNN "PACKAGE"
+	1    1400 1500
+	1    0    0    -1
+$EndComp
+Text Label 700  1600 2    50   ~ 0
+Gate1
+Text Label 4150 2050 2    50   ~ 0
+Gate1
+Text Label 2100 1600 0    50   ~ 0
+Drain1
+Text Label 3950 1750 0    50   ~ 0
+Drain1
+Text Label 2100 1700 0    50   ~ 0
+Source1
+Text Label 4350 1750 1    50   ~ 0
+Source1
+$Comp
+L MTP3055VL:MTP3055VL Q?
+U 1 1 60AC0CD1
+P 1400 2250
+F 0 "Q?" H 1400 2520 50  0000 C CNN
+F 1 "MTP3055VL" H 1400 2429 50  0000 C CNN
+F 2 "TO254P483X1016X2222-3P" H 1400 2250 50  0001 L BNN
+F 3 "" H 1400 2250 50  0001 L BNN
+F 4 "MTP3055VL" H 1400 2250 50  0001 L BNN "MPN"
+F 5 "18C7756" H 1400 2250 50  0001 L BNN "OC_NEWARK"
+F 6 "1845563" H 1400 2250 50  0001 L BNN "OC_FARNELL"
+F 7 "Fairchild" H 1400 2250 50  0001 L BNN "SUPPLIER"
+F 8 "TO-220" H 1400 2250 50  0001 L BNN "PACKAGE"
+	1    1400 2250
+	1    0    0    -1
+$EndComp
+Text Label 700  2350 2    50   ~ 0
+Gate2
+Text Label 2100 2350 0    50   ~ 0
+Drain2
+Text Label 2100 2450 0    50   ~ 0
+Source2
+Text Label 4150 4550 2    50   ~ 0
+Gate2
+Text Label 3950 4250 0    50   ~ 0
+Drain2
+Text Label 4350 4250 1    50   ~ 0
+Source2
 $EndSCHEMATC

Commit message: Put EVERYTHING in the 90x90 space
Ofc need to sort out the rats nest better. Nearly there
Parts:
- H1, H2, H3, H4: footprint MountingHole:MountingHole_3.5mm_Pad_TopBottom -> MountingHole:MountingHole_4mm_Pad
- Q5, Q6: renamed from Q?; footprint TO254P483X1016X2222-3P -> Package_TO_SOT_THT:TO-220-3_Vertical
Changed lines of the file:
@@
 F 0 "H1" V 9054 1600 50  0000 L CNN
 F 1 "MountingHole_Pad" V 9145 1600 50  0000 L CNN
-F 2 "MountingHole:MountingHole_3.5mm_Pad_TopBottom" H 9100 1450 50  0001 C CNN
+F 2 "MountingHole:MountingHole_4mm_Pad" H 9100 1450 50  0001 C CNN
 F 3 "~" H 9100 1450 50  0001 C CNN
 	1    9100 1450
@@
 F 0 "H2" V 9054 1800 50  0000 L CNN
 F 1 "MountingHole_Pad" V 9145 1800 50  0000 L CNN
-F 2 "MountingHole:MountingHole_3.5mm_Pad_TopBottom" H 9100 1650 50  0001 C CNN
+F 2 "MountingHole:MountingHole_4mm_Pad" H 9100 1650 50  0001 C CNN
 F 3 "~" H 9100 1650 50  0001 C CNN
 	1    9100 1650
@@
 F 0 "H3" V 9054 2000 50  0000 L CNN
 F 1 "MountingHole_Pad" V 9145 2000 50  0000 L CNN
-F 2 "MountingHole:MountingHole_3.5mm_Pad_TopBottom" H 9100 1850 50  0001 C CNN
+F 2 "MountingHole:MountingHole_4mm_Pad" H 9100 1850 50  0001 C CNN
 F 3 "~" H 9100 1850 50  0001 C CNN
 	1    9100 1850
@@
 F 0 "H4" V 9054 2200 50  0000 L CNN
 F 1 "MountingHole_Pad" V 9145 2200 50  0000 L CNN
-F 2 "MountingHole:MountingHole_3.5mm_Pad_TopBottom" H 9100 2050 50  0001 C CNN
+F 2 "MountingHole:MountingHole_4mm_Pad" H 9100 2050 50  0001 C CNN
 F 3 "~" H 9100 2050 50  0001 C CNN
 	1    9100 2050
@@
 	2950 6500 3200 6500
 $Comp
-L MTP3055VL:MTP3055VL Q?
+L MTP3055VL:MTP3055VL Q5
 U 1 1 60AA2630
 P 1400 1500
-F 0 "Q?" H 1400 1770 50  0000 C CNN
+F 0 "Q5" H 1400 1770 50  0000 C CNN
 F 1 "MTP3055VL" H 1400 1679 50  0000 C CNN
-F 2 "TO254P483X1016X2222-3P" H 1400 1500 50  0001 L BNN
+F 2 "Package_TO_SOT_THT:TO-220-3_Vertical" H 1400 1500 50  0001 L BNN
 F 3 "" H 1400 1500 50  0001 L BNN
 F 4 "MTP3055VL" H 1400 1500 50  0001 L BNN "MPN"
@@
 Source1
 $Comp
-L MTP3055VL:MTP3055VL Q?
+L MTP3055VL:MTP3055VL Q6
 U 1 1 60AC0CD1
 P 1400 2250
-F 0 "Q?" H 1400 2520 50  0000 C CNN
+F 0 "Q6" H 1400 2520 50  0000 C CNN
 F 1 "MTP3055VL" H 1400 2429 50  0000 C CNN
-F 2 "TO254P483X1016X2222-3P" H 1400 2250 50  0001 L BNN
+F 2 "Package_TO_SOT_THT:TO-220-3_Vertical" H 1400 2250 50  0001 L BNN
 F 3 "" H 1400 2250 50  0001 L BNN
 F 4 "MTP3055VL" H 1400 2250 50  0001 L BNN "MPN"

Commit message: Some connections
I hope this is ok
Parts:
- Q5, Q6: symbol MTP3055VL:MTP3055VL -> VLAD-rescue:MTP3055VL-MTP3055VL
Changed lines of the file:
@@
 EESchema Schematic File Version 4
-LIBS:VLAD-cache
 EELAYER 30 0
 EELAYER END
@@
 	2950 6500 3200 6500
 $Comp
-L MTP3055VL:MTP3055VL Q5
+L VLAD-rescue:MTP3055VL-MTP3055VL Q5
 U 1 1 60AA2630
 P 1400 1500
@@
 Source1
 $Comp
-L MTP3055VL:MTP3055VL Q6
+L VLAD-rescue:MTP3055VL-MTP3055VL Q6
 U 1 1 60AC0CD1
 P 1400 2250
