File: Hardware/PowerCircuitry.sch (KiCad schematic (older format))
At the start: 38 parts, among them J4 Conn_01x02_Male, J6 Conn_01x02_Male, Q5 Q_NMOS_GDS, Q6 Q_NMOS_GDS, Q7 Q_NMOS_GDS, U4 MAX40200AUK

Commit message: Need some THT - SMD changes
Inductors, capacitors, MAX1771CSA, the LED dudes and the ones next to the ESP
Parts:
- D2, D3: footprint Diode_THT:D_DO-34_SOD68_P7.62mm_Horizontal -> Diode_SMD:D_SOD-123F
Changed lines of the file:
@@
 F 0 "D2" H 3950 1216 50  0000 C CNN
 F 1 "D_Schottky" H 3950 1125 50  0000 C CNN
-F 2 "Diode_THT:D_DO-34_SOD68_P7.62mm_Horizontal" H 3950 1000 50  0001 C CNN
+F 2 "Diode_SMD:D_SOD-123F" H 3950 1000 50  0001 C CNN
 F 3 "~" H 3950 1000 50  0001 C CNN
 	1    3950 1000
@@
 F 0 "D3" H 3950 3716 50  0000 C CNN
 F 1 "D_Schottky" H 3950 3625 50  0000 C CNN
-F 2 "Diode_THT:D_DO-34_SOD68_P7.62mm_Horizontal" H 3950 3500 50  0001 C CNN
+F 2 "Diode_SMD:D_SOD-123F" H 3950 3500 50  0001 C CNN
 F 3 "~" H 3950 3500 50  0001 C CNN
 	1    3950 3500

Commit message: Executive decision to use THT capacitors
THT >>>>>>>>>>>> SMD
Parts:
- 12VBoostConverter1, 6VBoostConverter1: footprint footprints:max1771cpa&plus_ -> iclr:MAX1771CSA&plus_

Commit message: Traccs done, meme time
Need to fix the silkscreen stuff for the components and also the back silkscreen memes etc.
Parts:
- 12VBoostConverter1, 6VBoostConverter1: value max1771cpa+ -> max1771csa+
Changed lines of the file:
@@
 P 4150 2050
 F 0 "12VBoostConverter1" H 5350 2437 60  0000 C CNN
-F 1 "max1771cpa+" H 5350 2331 60  0000 C CNN
+F 1 "max1771csa+" H 5350 2331 60  0000 C CNN
 F 2 "iclr:MAX1771CSA&plus_" H 5350 2290 60  0001 C CNN
 F 3 "" H 4150 2050 60  0000 C CNN
@@
 P 4150 4550
 F 0 "6VBoostConverter1" H 5350 4937 60  0000 C CNN
-F 1 "max1771cpa+" H 5350 4831 60  0000 C CNN
+F 1 "max1771csa+" H 5350 4831 60  0000 C CNN
 F 2 "iclr:MAX1771CSA&plus_" H 5350 4790 60  0001 C CNN
 F 3 "" H 4150 4550 60  0000 C CNN
